Commit message: minimal properties implementation

File: tests/data/property_test_expected.xacro (robot description, xacro)
@@ -1,5 +1,4 @@
 <?xml version="1.0"?>
 <robot name="test_robot" xmlns:xacro="http://www.ros.org/wiki/xacro">
-    <property name="width" value="0.5"/>
-    <box size="${width}"/>
+    <box size="0.5"/>
 </robot>

File: tests/data/property_test_nested.xacro (robot description, xacro)
@@ -1,5 +1,6 @@
 <?xml version="1.0"?>
 <robot name="test_robot" xmlns:xacro="http://www.ros.org/wiki/xacro">
-    <property name="width" value="0.5"/>
-    <box size="${width}"/>
+    <property name="x" value="1"/>
+    <property name="y" value="${x}"/>
+    <point coord="${y}"/>
 </robot>

File: tests/data/property_test_nested_expected.xacro (robot description, xacro)
@@ -1,5 +1,4 @@
 <?xml version="1.0"?>
 <robot name="test_robot" xmlns:xacro="http://www.ros.org/wiki/xacro">
-    <property name="width" value="0.5"/>
-    <box size="${width}"/>
+    <point coord="1"/>
 </robot>
