Commit message: formatting xml

File: tests/data/include_test.xacro (robot description, xacro)
@@ -1,5 +1,5 @@
 <?xml version="1.0"?>
 <robot name="test_robot" xmlns:xacro="http://www.ros.org/wiki/xacro">
-    <xacro:include filename="include_test_component.xacro"/>
-    <link name="additional_link"/>
+ <xacro:include filename="include_test_component.xacro"/>
+ <link name="additional_link"/>
 </robot>

File: tests/data/include_test_component.xacro (robot description, xacro)
@@ -1,10 +1,10 @@
 <?xml version="1.0"?>
 <robot xmlns:xacro="http://www.ros.org/wiki/xacro">
-    <link name="base_link">
-        <visual>
-            <geometry>
-                <cylinder length="0.6" radius="0.2"/>
-            </geometry>
-        </visual>
-    </link>
+ <link name="base_link">
+  <visual>
+   <geometry>
+    <cylinder length="0.6" radius="0.2"/>
+   </geometry>
+  </visual>
+ </link>
 </robot>

File: tests/data/include_test_directory.xacro (robot description, xacro)
@@ -1,5 +1,5 @@
 <?xml version="1.0"?>
 <robot name="test_robot" xmlns:xacro="http://www.ros.org/wiki/xacro">
-  <xacro:include filename="include/include_test_directory_component.xacro"/>
-    <link name="additional_link"/>
+ <xacro:include filename="include/include_test_directory_component.xacro"/>
+ <link name="additional_link"/>
 </robot>

File: tests/data/include_test_directory_expected.xacro (robot description, xacro)
@@ -1,11 +1,11 @@
 <?xml version="1.0"?>
 <robot name="test_robot" xmlns:xacro="http://www.ros.org/wiki/xacro">
-    <link name="base_link">
-        <visual>
-            <geometry>
-                <cylinder length="0.6" radius="0.2"/>
-            </geometry>
-        </visual>
-    </link>
-    <link name="additional_link"/>
+ <link name="base_link">
+  <visual>
+   <geometry>
+    <cylinder length="0.6" radius="0.2"/>
+   </geometry>
+  </visual>
+ </link>
+ <link name="additional_link"/>
 </robot>

File: tests/data/include_test_multi_arms.xacro (robot description, xacro)
@@ -1,4 +1,4 @@
 <robot xmlns:xacro="http://www.ros.org/wiki/xacro">
-    <link name="arm_left_link"/>
-    <link name="arm_right_link"/>
+ <link name="arm_left_link"/>
+ <link name="arm_right_link"/>
 </robot>

File: tests/data/include_test_multi_base.xacro (robot description, xacro)
@@ -1,5 +1,5 @@
 <?xml version="1.0"?>
 <robot name="test_robot" xmlns:xacro="http://www.ros.org/wiki/xacro">
-  <xacro:include filename="include_test_multi_wheels.xacro"/>
-  <xacro:include filename="include_test_multi_arms.xacro"/>
+ <xacro:include filename="include_test_multi_wheels.xacro"/>
+ <xacro:include filename="include_test_multi_arms.xacro"/>
 </robot>

File: tests/data/include_test_multi_expected.xacro (robot description, xacro)
@@ -1,7 +1,7 @@
 <?xml version="1.0"?>
 <robot name="test_robot" xmlns:xacro="http://www.ros.org/wiki/xacro">
-    <link name="wheel_front_right"/>
-    <link name="wheel_front_left"/>
-    <link name="arm_left_link"/>
-    <link name="arm_right_link"/>
+ <link name="wheel_front_right"/>
+ <link name="wheel_front_left"/>
+ <link name="arm_left_link"/>
+ <link name="arm_right_link"/>
 </robot>

File: tests/data/include_test_multi_wheels.xacro (robot description, xacro)
@@ -1,5 +1,5 @@
 <?xml version="1.0"?>
 <robot xmlns:xacro="http://www.ros.org/wiki/xacro">
-    <link name="wheel_front_right"/>
-    <link name="wheel_front_left"/>
+ <link name="wheel_front_right"/>
+ <link name="wheel_front_left"/>
 </robot>

File: tests/data/include_test_nested_arm.xacro (robot description, xacro)
@@ -1,6 +1,6 @@
 <?xml version="1.0"?>
 <robot xmlns:xacro="http://www.ros.org/wiki/xacro">
-    <link name="arm_base"/>
-    <link name="arm_link_1"/>
-    <xacro:include filename="include_test_nested_hand.xacro"/>
+ <link name="arm_base"/>
+ <link name="arm_link_1"/>
+ <xacro:include filename="include_test_nested_hand.xacro"/>
 </robot>

File: tests/data/include_test_nested_base.xacro (robot description, xacro)
@@ -1,4 +1,4 @@
 <?xml version="1.0"?>
 <robot name="test_robot" xmlns:xacro="http://www.ros.org/wiki/xacro">
-    <xacro:include filename="include_test_nested_arm.xacro"/>
+ <xacro:include filename="include_test_nested_arm.xacro"/>
 </robot>

File: tests/data/include_test_nested_expected.xacro (robot description, xacro)
@@ -1,8 +1,8 @@
 <?xml version="1.0"?>
 <robot name="test_robot" xmlns:xacro="http://www.ros.org/wiki/xacro">
-    <link name="arm_base"/>
-    <link name="arm_link_1"/>
-    <link name="hand_base"/>
-    <link name="hand_finger_1"/>
-    <link name="hand_finger_2"/>
+ <link name="arm_base"/>
+ <link name="arm_link_1"/>
+ <link name="hand_base"/>
+ <link name="hand_finger_1"/>
+ <link name="hand_finger_2"/>
 </robot>

File: tests/data/include_test_nested_hand.xacro (robot description, xacro)
@@ -1,6 +1,6 @@
 <?xml version="1.0"?>
 <robot xmlns:xacro="http://www.ros.org/wiki/xacro">
-    <link name="hand_base"/>
-    <link name="hand_finger_1"/>
-    <link name="hand_finger_2"/>
+ <link name="hand_base"/>
+ <link name="hand_finger_1"/>
+ <link name="hand_finger_2"/>
 </robot>

File: tests/data/property_test_base.xacro (robot description, xacro)
@@ -1,5 +1,5 @@
 <?xml version="1.0"?>
 <robot name="test_robot" xmlns:xacro="http://www.ros.org/wiki/xacro">
-    <property name="width" value="0.5"/>
-    <box size="${width}"/>
+ <property name="width" value="0.5"/>
+ <box size="${width}"/>
 </robot>

File: tests/data/property_test_expected.xacro (robot description, xacro)
@@ -1,4 +1,4 @@
 <?xml version="1.0"?>
 <robot name="test_robot" xmlns:xacro="http://www.ros.org/wiki/xacro">
-    <box size="0.5"/>
+ <box size="0.5"/>
 </robot>

File: tests/data/property_test_nested.xacro (robot description, xacro)
@@ -1,6 +1,6 @@
 <?xml version="1.0"?>
 <robot name="test_robot" xmlns:xacro="http://www.ros.org/wiki/xacro">
-    <property name="x" value="1"/>
-    <property name="y" value="${x}"/>
-    <point coord="${y}"/>
+ <property name="x" value="1"/>
+ <property name="y" value="${x}"/>
+ <point coord="${y}"/>
 </robot>

File: tests/data/property_test_nested_expected.xacro (robot description, xacro)
@@ -1,4 +1,4 @@
 <?xml version="1.0"?>
 <robot name="test_robot" xmlns:xacro="http://www.ros.org/wiki/xacro">
-    <point coord="1"/>
+ <point coord="1"/>
 </robot>
