Commit message: property testing basics

File: tests/data/include_test_multi_arms.xacro (robot description, xacro)
@@ -1,2 +1,3 @@
+<?xml version="1.0"?>
 <robot xmlns:xacro="http://www.ros.org/wiki/xacro">
  <link name="arm_left_link"/>

File: tests/data/property_test_attributes_expected.xacro (robot description, xacro)
@@ -1,4 +1,4 @@
 <?xml version="1.0"?>
 <robot name="test_robot" xmlns:xacro="http://www.ros.org/wiki/xacro">
- <box size="0.5 1.0 0.3"/>
+ <link name="arm_link"/>
 </robot>

File: tests/data/property_test_multi_substitution_expected.xacro (robot description, xacro)
@@ -1,4 +1,4 @@
 <?xml version="1.0"?>
 <robot name="test_robot" xmlns:xacro="http://www.ros.org/wiki/xacro">
- <box size="0.5 1.0 0.3"/>
+ <elem value="prefix_first_middle_second_suffix"/>
 </robot>

File: tests/data/property_test_multiple.xacro (robot description, xacro)
@@ -1,2 +1,3 @@
+<?xml version="1.0"?>
 <robot name="test_robot" xmlns:xacro="http://www.ros.org/wiki/xacro">
  <xacro:property name="width" value="0.5"/>

File: tests/data/property_test_multiple_out_of_order.xacro (robot description, xacro)
@@ -1,2 +1,3 @@
+<?xml version="1.0"?>
 <robot name="test_robot" xmlns:xacro="http://www.ros.org/wiki/xacro">
  <xacro:property name="base" value="0.5"/>

File: tests/data/property_test_multiple_out_of_order_expected.xacro (robot description, xacro)
@@ -1,2 +1,3 @@
+<?xml version="1.0"?>
 <robot name="test_robot" xmlns:xacro="http://www.ros.org/wiki/xacro">
  <box size="0.5 2"/>
